File: minidexed-hat.kicad_pcb (KiCad board)
At the start: 2 copper layers, 56 x 65 mm, 14 parts, among them J1 MIDI, J2 Line out, J3 RPi_GPIO, J4 Encoder, J5 9-12V, J6 LCD, J7 I2C, U1 PCM5102_Module

Commit message: Add text
Other:
- board text added: "12VDC"
- board text added: "MiniDexed Hat for Raspberry Pi Rev. 1 Paul Battley 2022 po-ru.com/pcb/minidexed"
- board text removed: "9-12VDC"
Changed lines of the file:
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@@
+    (effects (font (size 0.8128 0.8128) (thickness 0.1524)) (justify left))
+  )
+  (gr_text "MiniDexed Hat for Raspberry Pi Rev. 1\nPaul Battley 2022\npo-ru.com/pcb/minidexed" (at 58.5 53) (layer "F.SilkS")
     (effects (font (size 0.8128 0.8128) (thickness 0.1524)) (justify left))
   )
@@
     (effects (font (size 0.8128 0.8128) (thickness 0.1524)))
   )
-  (gr_text "9-12VDC" (at 94.5 56) (layer "F.SilkS")
+  (gr_text "12VDC" (at 94.5 56) (layer "F.SilkS")
     (effects (font (size 0.8128 0.8128) (thickness 0.1524)))
   )

Commit message: Add placeholder for order number
Other:
- board text added: "JLCJLCJLCJLC"
Changed lines of the file:
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@@
   (gr_arc (start 103 50) (mid 105.12132 50.87868) (end 106 53) (layer "Edge.Cuts") (width 0.15))
   (gr_arc (start 53 115) (mid 50.87868 114.12132) (end 50 112) (layer "Edge.Cuts") (width 0.15))
+  (gr_text "JLCJLCJLCJLC" (at 80.5 54) (layer "B.SilkS")
+    (effects (font (size 0.8128 0.8128) (thickness 0.1524)) (justify mirror))
+  )
   (gr_text "RS" (at 62.23 96.52) (layer "F.SilkS")
     (effects (font (size 0.8128 0.8128) (thickness 0.1524)) (justify left))
